Commit message: Support wheeled arm synthetic camera capture
Allow mock_cameras to run with real wheeled arm feedback by skipping camera connect/read/disconnect and generating synthetic observations. Update the wheeled arm default ROS2 camera size and tighten PICO wrist joint limits, with regression coverage for the real-robot synthetic-camera path.

File: src/lerobot/teleoperators/wheeled_arm_pico/assets/wheeled_robot_sim/urdf/real_robot.urdf (robot description, URDF)
Before this commit: robot real_robot, 28 links, 27 joints
Joints:
- joint AR5-5_07L-W4C4A2_joint_6: limit lower=-1.0472 upper=1.0472 effort=19 velocity=4.1887902047863905 -> lower=-0.9 upper=0.9 effort=19 velocity=4.1887902047863905
- joint AR5-5_07L-W4C4A2_joint_7: limit lower=-1.0472 upper=1.0472 effort=19 velocity=4.1887902047863905 -> lower=-0.9 upper=0.9 effort=19 velocity=4.1887902047863905
- joint AR5-5_07R-W4C4A2_joint_6: limit lower=-1.0472 upper=1.0472 effort=19 velocity=4.1887902047863905 -> lower=-0.9 upper=0.9 effort=19 velocity=4.1887902047863905
- joint AR5-5_07R-W4C4A2_joint_7: limit lower=-1.0472 upper=1.0472 effort=19 velocity=4.1887902047863905 -> lower=-0.9 upper=0.9 effort=19 velocity=4.1887902047863905
